Commit message: fixed typos

File: robot_descriptions/marcel_arm/marcel_arm.urdf (robot description, URDF)
Before this commit: robot seven_link_robot, 9 links, 8 joints
Links:
- link link0: geometry collision mesh filename=package://link0.dae scale=0.001 0.001 0.001; visual mesh filename=package://link0.dae scale=0.001 0.001 0.001
- link link1: geometry collision mesh filename=package://link1.dae scale=0.001 0.001 0.001; visual mesh filename=package://link1.dae scale=0.001 0.001 0.001
- link link2: geometry collision mesh filename=package://link2.dae scale=0.001 0.001 0.001; visual mesh filename=package://link2.dae scale=0.001 0.001 0.001
- link link3: geometry collision mesh filename=package://link3.dae scale=0.001 0.001 0.001; visual mesh filename=package://link3.dae scale=0.001 0.001 0.001
- link link4: geometry collision mesh filename=package://link4.dae scale=0.001 0.001 0.001; visual mesh filename=package://link4.dae scale=0.001 0.001 0.001
- link link5: geometry collision mesh filename=package://link5.dae scale=0.001 0.001 0.001; visual mesh filename=package://link5.dae scale=0.001 0.001 0.001
- link link6: geometry collision mesh filename=package://link6.dae scale=0.001 0.001 0.001; visual mesh filename=package://link6.dae scale=0.001 0.001 0.001
Joints:
- joint joint5: axis 0 1 0 -> 0 -1 0; limit lower=-1.39626 upper=0.0872665 effort=100 velocity=1 -> lower=-0.0872665 upper=1.39626 effort=100 velocity=1

File: robot_descriptions/marcel_plus_wx250s/urdf/bimanual.urdf (robot description, URDF)
Before this commit: robot wx250s, 23 links, 22 joints
Joints:
- joint joint5: axis 0 1 0 -> 0 -1 0; limit lower=-1.39626 upper=0.0872665 effort=100 velocity=1 -> lower=-0.0872665 upper=1.39626 effort=100 velocity=1
